File: hw/creeper/creeper.kicad_pcb (KiCad board)
At the start: 2 copper layers, 35 x 35 mm, 29 parts, among them J1 TC2030_AVR, J2 Conn_01x06_Pin, SW1 EG1213, U1 ATtiny85V-10SU, U2 IIS328DQTR

Commit message: ci(kibot): add KiBot configuration and fix some minor issues
Parts:
- renumbered QR***** to QR1, REF** to REF**3
Changed lines of the file:
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@@
 		(descr "Mounting Hole 2.2mm, M2, generated by kicad-footprint-generator mountinghole.py")
 		(tags "mountinghole M2 DIN965")
-		(property "Reference" "REF**"
+		(property "Reference" "REF**3"
 			(at 0 -2.85 0)
 			(layer "F.SilkS")
@@
 		(layer "B.Cu")
 		(at 129.47 76.14)
-		(property "Reference" "QR*****"
+		(property "Reference" "QR1"
 			(at 0 -5.375 180)
 			(layer "B.SilkS")
