File: hw/creeper/creeper.kicad_sch (KiCad schematic)
At the start: 25 parts, among them J1 TC2030_AVR, J2 Conn_01x06_Pin, SW1 EG1213, U1 ATtiny85V-10SU, U2 IIS328DQTR

Commit message: ci(kibot): add KiBot configuration and fix some minor issues
Parts:
- BT1: MANUFACTURER (none) -> Keystone Electronics
- C_ACC1, C_MCU1, C_SWI1: MANUFACTURER (none) -> KEMET
- C_PWR1: MANUFACTURER (none) -> Murata Electronics
- D1, D2: MANUFACTURER (none) -> ams-OSRAM USA INC.
- RPU_CS1, RPU_INT1, RPU_RST1, RPU_SCL1, RPU_SDA1, R_BUZ1, R_LED1, R_LED2: MANUFACTURER (none) -> Vishay Dale
- SW1: MANUFACTURER (none) -> E-Switch
- U1: MANUFACTURER (none) -> Microchip Technology
- U2: MANUFACTURER (none) -> ST Microelectronics
- U3: MANUFACTURER (none) -> Nexperia USA Inc.
Changed lines of the file:
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@@
 			)
 		)
-		(property "MANUFACTURER" ""
+		(property "MANUFACTURER" "Vishay Dale"
 			(at 48.26 88.9 90)
 			(effects
@@
 			)
 		)
-		(property "MANUFACTURER" ""
+		(property "MANUFACTURER" "Nexperia USA Inc."
 			(at 151.13 53.34 0)
 			(effects
@@
 			)
 		)
-		(property "MANUFACTURER" ""
+		(property "MANUFACTURER" "KEMET"
 			(at 105.41 38.1 90)
 			(effects
@@
 			)
 		)
-		(property "MANUFACTURER" ""
+		(property "MANUFACTURER" "Vishay Dale"
 			(at 96.52 85.09 0)
 			(effects
@@
 			)
 		)
-		(property "MANUFACTURER" ""
+		(property "MANUFACTURER" "KEMET"
 			(at 78.74 171.45 90)
 			(effects
@@
 			)
 		)
-		(property "MANUFACTURER" ""
+		(property "MANUFACTURER" "Vishay Dale"
 			(at 119.38 60.96 90)
 			(effects
@@
 			)
 		)
-		(property "MANUFACTURER" ""
+		(property "MANUFACTURER" "Vishay Dale"
 			(at 142.24 88.9 0)
 			(effects
@@
 			)
 		)
-		(property "MANUFACTURER" ""
+		(property "MANUFACTURER" "ams-OSRAM USA INC."
 			(at 106.68 91.44 0)
 			(effects
@@
 			)
 		)
-		(property "MANUFACTURER" ""
+		(property "MANUFACTURER" "ams-OSRAM USA INC."
 			(at 96.52 91.44 0)
 			(effects
@@
 			)
 		)
-		(property "MANUFACTURER" ""
+		(property "MANUFACTURER" "Keystone Electronics"
 			(at 50.8 63.5 0)
 			(effects
@@
 			)
 		)
-		(property "MANUFACTURER" ""
+		(property "MANUFACTURER" "Murata Electronics"
 			(at 39.37 62.23 0)
 			(effects
@@
 			)
 		)
-		(property "MANUFACTURER" ""
+		(property "MANUFACTURER" "Vishay Dale"
 			(at 157.48 88.9 0)
 			(effects
@@
 			)
 		)
-		(property "MANUFACTURER" ""
+		(property "MANUFACTURER" "Vishay Dale"
 			(at 82.55 54.61 90)
 			(effects
@@
 			)
 		)
-		(property "MANUFACTURER" ""
+		(property "MANUFACTURER" "Vishay Dale"
 			(at 38.1 153.67 0)
 			(effects
@@
 			)
 		)
-		(property "MANUFACTURER" ""
+		(property "MANUFACTURER" "E-Switch"
 			(at 57.15 40.64 0)
 			(effects
@@
 			)
 		)
-		(property "MANUFACTURER" ""
+		(property "MANUFACTURER" "KEMET"
 			(at 158.75 38.1 90)
 			(effects
@@
 			)
 		)
-		(property "MANUFACTURER" ""
+		(property "MANUFACTURER" "Microchip Technology"
 			(at 101.6 53.34 0)
 			(effects
@@
 			)
 		)
-		(property "MANUFACTURER" ""
+		(property "MANUFACTURER" "Vishay Dale"
 			(at 106.68 85.09 0)
 			(effects
@@
 			)
 		)
-		(property "MANUFACTURER" ""
+		(property "MANUFACTURER" "ST Microelectronics"
 			(at 55.88 158.75 0)
 			(effects
